Commit message: Changed Differential drive sim, setup script, and URDF

File: midterm/en613_control/urdf/basic_robot.urdf (robot description, URDF)
Before this commit: robot rockman, 5 links, 4 joints
Joints:
- removed joint base_to_lidar_dome
- added joint chassis_to_lidar_dome: type fixed, parent chassis, child lidar_dome, origin xyz=0.3 0 0.0375 rpy=0 0 -1.5707
- joint base_to_chassis: origin xyz=0 0 0 rpy=0 0 1.5707 -> xyz=0 0 0.4 rpy=0 0 1.5707
- joint base_to_right_wheel: axis (none) -> 0 0 1; limit lower=0.0 upper=0.548 effort=1000.0 velocity=0.5 -> (none); type revolute -> continuous
- joint chassis_to_left_wheel: axis (none) -> 0 0 1; limit lower=0.0 upper=0.548 effort=1000.0 velocity=0.5 -> (none); type revolute -> continuous

Commit message: Small update to diffdrive_sim, added TF to RVIZ config, and changed the URDF to remove the base frame

File: midterm/en613_control/urdf/basic_robot.urdf (robot description, URDF)
Before this commit: robot rockman, 5 links, 4 joints
Links:
- removed link base
Joints:
- removed joint base_to_chassis

Commit message: Fixed the joints not spinning

File: midterm/en613_control/urdf/basic_robot.urdf (robot description, URDF)
Before this commit: robot rockman, 4 links, 3 joints
Joints:
- removed joint base_to_right_wheel
- added joint chassis_to_right_wheel: type continuous, parent chassis, child right_wheel, origin xyz=0 -0.4375 0 rpy=-1.5707 0 0, axis 0 0 1

Commit message: The PID kinda works :(

File: midterm/en613_control/urdf/basic_robot.urdf (robot description, URDF)
Before this commit: robot rockman, 4 links, 3 joints
Joints:
- joint chassis_to_lidar_dome: origin xyz=0.3 0 0.0375 rpy=0 0 -1.5707 -> xyz=0.3 0 0.0375 rpy=0 0 0
